File: template/stencil/stencil.kicad_pcb (KiCad board)
At the start: 4 copper layers, 280 x 380 mm, 3 parts

Commit message: Update stencil template
Other:
- board text added: "280 x 380 -> 200 x 310"
- board text removed: "280 x 380 → 200 x 310"
Changed lines of the file:
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@@
 		(layer "Edge.Cuts")
-	)
-	(gr_line
-		(start 140 345)
-		(end 140 35)
-		(stroke
-			(width 0.2)
-			(type dash)
-		)
-		(locked yes)
-		(layer "F.Fab")
 	)
 	(gr_rect
@@
 	)
 	(gr_line
+		(start 140 345)
+		(end 140 35)
+		(stroke
+			(width 0.2)
+			(type dash)
+		)
+		(locked yes)
+		(layer "F.Fab")
+	)
+	(gr_line
 		(start 240 190)
 		(end 40 190)
@@
 		(locked yes)
 		(layer "F.Fab")
-	)
-	(gr_text "280 x 380 → 200 x 310"
-		(locked yes)
-		(at 221.5 377.25 0)
-		(layer "F.Fab")
-		(effects
-			(font
-				(size 3 3)
-				(thickness 0.6)
-				(bold yes)
-			)
-			(justify left bottom)
-		)
 	)
 	(gr_text "V2"
@@
 		)
 	)
+	(gr_text "280 x 380 -> 200 x 310"
+		(locked yes)
+		(at 212.5 373.75 0)
+		(layer "F.Fab")
+		(effects
+			(font
+				(size 3 3)
+				(thickness 0.6)
+				(bold yes)
+			)
+			(justify left bottom)
+		)
+	)

Commit message: Update stencil
Parts:
- moved FID101 5.00 mm to (50.0, 340.0)
- moved FID102 5.00 mm to (230.0, 340.0)
- moved FID103 5.00 mm to (50.0, 40.0)
Other:
- board text added: "280 x 380 -> 200 x 320"
- board text removed: "280 x 380 -> 200 x 310"
Changed lines of the file:
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@@
 	(paper "User" 280 380)
 	(title_block
-		(date "2026-01-10")
+		(date "2026-01-28")
 	)
 	(layers
@@
 		(allow_soldermask_bridges_in_footprints no)
 		(tenting front back)
-		(aux_axis_origin 40 345)
-		(grid_origin 40 345)
+		(aux_axis_origin 40 350)
+		(grid_origin 40 350)
 		(pcbplotparams
 			(layerselection 0x00000000_00000000_55555555_55557500)
@@
 	(footprint "V2_Fiducial:Fiducial_0.5mm_Mask1mm_Paste"
 		(layer "F.Cu")
-		(at 230 335)
+		(at 230 340)
 		(descr "Circular Fiducial, 0.5mm bare copper, 1mm soldermask opening (Level C)")
 		(tags "fiducial")
@@
 	(footprint "V2_Fiducial:Fiducial_0.5mm_Mask1mm_Paste"
 		(layer "F.Cu")
-		(at 50 45)
+		(at 50 40)
 		(descr "Circular Fiducial, 0.5mm bare copper, 1mm soldermask opening (Level C)")
 		(tags "fiducial")
@@
 	(footprint "V2_Fiducial:Fiducial_0.5mm_Mask1mm_Paste"
 		(layer "F.Cu")
-		(at 50 335)
+		(at 50 340)
 		(descr "Circular Fiducial, 0.5mm bare copper, 1mm soldermask opening (Level C)")
 		(tags "fiducial")
@@
 	)
 	(gr_rect
-		(start 40 35)
-		(end 240 345)
+		(start 40 30)
+		(end 240 350)
 		(stroke
 			(width 0.2)
@@
 	)
 	(gr_line
-		(start 140 345)
-		(end 140 35)
+		(start 140 350)
+		(end 140 30)
 		(stroke
 			(width 0.2)
@@
 		)
 	)
-	(gr_text "280 x 380 -> 200 x 310"
+	(gr_text "280 x 380 -> 200 x 320"
 		(locked yes)
 		(at 212.5 373.75 0)
@@
 	)
 	(embedded_fonts no)
+	(embedded_files
+		(file
+			(name "V2_A4_Empty.kicad_wks")
+			(type worksheet)
+			(data |KLUv/SDtTQQA8kcaGHDNA0DI0YHeJkZJsFFVHWPECK8T+nf7Ruut19T/Wjj1lcRtZEY9sbORjzTz
+				BIaRKX941NSZJ0BmPfl9qd8ptZzn+0ZINNlsfT9aMk5jtv60TTtxar2BmQMgAoxWv7Yhp9ZdInlM
+				wxcXCyAQIoF8eJTajUPCXqolYFHFD/FgziWduMYHggI=|
+			)
+			(checksum "00BCE598336E5951A5D0C187D2E96FE2")
+		)
+	)
 )

Commit message: Update stencil template
Parts:
- FID101, FID102, FID103: value Fiducial -> Fiducial_Paste
Changed lines of the file:
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@@
 	(paper "User" 280 380)
 	(title_block
-		(date "2026-01-28")
+		(date "2026-02-10")
 	)
 	(layers
@@
 			)
 		)
-		(property "Value" "Fiducial"
+		(property "Value" "Fiducial_Paste"
 			(at 0 1.5 0)
 			(layer "F.Fab")
@@
 			)
 		)
-		(property "Description" "Fiducial Marker"
+		(property "Description" ""
 			(at 0 0 0)
 			(unlocked yes)
@@
 			)
 		)
-		(property "Value" "Fiducial"
+		(property "Value" "Fiducial_Paste"
 			(at 0 1.5 0)
 			(layer "F.Fab")
@@
 			)
 		)
-		(property "Description" "Fiducial Marker"
+		(property "Description" ""
 			(at 0 0 0)
 			(unlocked yes)
@@
 			)
 		)
-		(property "Value" "Fiducial"
+		(property "Value" "Fiducial_Paste"
 			(at 0 1.5 0)
 			(layer "F.Fab")
@@
 			)
 		)
-		(property "Description" "Fiducial Marker"
-			(at 0 0 0)
-			(unlocked yes)
+		(property "Description" ""
+			(at 0 0 0)
+			(unlocked yes)
