File: template/stencil/stencil.kicad_pcb (KiCad board)
At the start: 4 copper layers, 280 x 380 mm, 3 parts

Commit message: Update stencil template
Other:
- board text added: "${REVISION} @{if(${REVISION} != ${ISSUE_DATE}, {dblquote}(${ISSUE_DATE}){dblquote}, {dblquote}{dblquote})}"
- board text removed: "V2"
Changed lines of the file:
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@@
 	(paper "User" 280 380)
 	(title_block
-		(date "2026-03-25")
-		(rev "2026-03-21")
+		(date "2026-04-24")
+		(rev "2026-04-24")
 	)
 	(layers
@@
 				(color "Black")
 				(thickness 0.01)
-			)
-			(layer "dielectric 4"
-				(type "Bottom Silk Screen")
-				(thickness 0)
-				(material "FR4")
-				(epsilon_r 4.5)
-				(loss_tangent 0.02)
 			)
 			(copper_finish "HAL lead-free")
@@
 		(layer "F.Fab")
 	)
-	(gr_text "V2"
+	(gr_text "${REVISION} @{if(${REVISION} !=  ${ISSUE_DATE}, {dblquote}(${ISSUE_DATE}){dblquote}, {dblquote}{dblquote})}\n\n"
 		(at 7.75 8.25 0)
 		(layer "F.Fab")

Commit message: Fix Revision - Issue comparison
Other:
- board text added: "${REVISION} @{if({dblquote}${REVISION}{dblquote} != {dblquote}${ISSUE_DATE}{dblquote}, {dblquote}(${ISSUE_DATE}){dblquote}, {dblquote}{dblquote})}"
- board text removed: "${REVISION} @{if(${REVISION} != ${ISSUE_DATE}, {dblquote}(${ISSUE_DATE}){dblquote}, {dblquote}{dblquote})}"
Changed lines of the file:
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@@
 	(paper "User" 280 380)
 	(title_block
-		(date "2026-04-24")
-		(rev "2026-04-24")
+		(date "2026-06-06")
+		(rev "2026-06-06")
 	)
 	(layers
@@
 		(layer "F.Fab")
 	)
-	(gr_text "${REVISION} @{if(${REVISION} !=  ${ISSUE_DATE}, {dblquote}(${ISSUE_DATE}){dblquote}, {dblquote}{dblquote})}\n\n"
+	(gr_text "${REVISION} @{if({dblquote}${REVISION}{dblquote} !=  {dblquote}${ISSUE_DATE}{dblquote}, {dblquote}(${ISSUE_DATE}){dblquote}, {dblquote}{dblquote})}"
 		(at 7.75 8.25 0)
 		(layer "F.Fab")
