File: template/stencil/stencil.kicad_pcb (KiCad board)
At the start: 4 copper layers, 280 x 380 mm, 3 parts

Commit message: Update stencil
Other:
- board text added: "1:1 please. No changes. Do NOT remove any fiducials. Thanks!"
Changed lines of the file:
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@@
 	(generator_version "10.0")
 	(general
-		(thickness 1.6062)
+		(thickness 1.6222)
 		(legacy_teardrops no)
 	)
 	(paper "User" 280 380)
 	(title_block
-		(date "2026-06-06")
-		(rev "2026-06-06")
+		(date "2026-07-18")
+		(rev "2026-07-18")
 	)
 	(layers
@@
 		(13 "F.Paste" user)
 		(5 "F.SilkS" user "F.Silkscreen")
+		(7 "B.SilkS" user "B.Silkscreen")
 		(1 "F.Mask" user)
 		(3 "B.Mask" user)
+		(19 "Cmts.User" user "User.Comments")
 		(25 "Edge.Cuts" user)
 		(27 "Margin" user)
@@
 		(29 "B.CrtYd" user "B.Courtyard")
 		(35 "F.Fab" user)
+		(33 "B.Fab" user)
 	)
 	(setup
@@
 			(layer "F.SilkS"
 				(type "Top Silk Screen")
-				(color "White")
 			)
 			(layer "F.Paste"
@@
 			(layer "F.Mask"
 				(type "Top Solder Mask")
-				(color "Black")
-				(thickness 0.01)
+				(thickness 0.018)
 			)
 			(layer "F.Cu"
@@
 			(layer "B.Mask"
 				(type "Bottom Solder Mask")
-				(color "Black")
-				(thickness 0.01)
+				(thickness 0.018)
+			)
+			(layer "B.SilkS"
+				(type "Bottom Silk Screen")
 			)
 			(copper_finish "HAL lead-free")
@@
 		(grid_origin 40 350)
 		(pcbplotparams
-			(layerselection 0x00000000_00000000_55555555_55557500)
+			(layerselection 0x00000000_00000000_55555555_555d7500)
 			(plot_on_all_layers_selection 0x00000000_00000000_00000000_00000000)
 			(disableapertmacros no)
@@
 	)
 	(gr_rect
-		(start 0 0)
-		(end 280 380)
-		(stroke
-			(width 0.1)
-			(type solid)
-		)
-		(fill no)
-		(layer "Edge.Cuts")
-	)
-	(gr_rect
 		(start 40 30)
 		(end 240 350)
+		(radius 3)
 		(stroke
 			(width 0.2)
@@
 		(fill no)
 		(locked yes)
-		(layer "F.Fab")
+		(layer "Cmts.User")
 	)
 	(gr_line
@@
 		)
 		(locked yes)
-		(layer "F.Fab")
+		(layer "Cmts.User")
 	)
 	(gr_line
@@
 		)
 		(locked yes)
-		(layer "F.Fab")
+		(layer "Cmts.User")
+	)
+	(gr_rect
+		(start 0 0)
+		(end 280 380)
+		(stroke
+			(width 0.1)
+			(type solid)
+		)
+		(fill no)
+		(layer "Edge.Cuts")
 	)
 	(gr_text "${REVISION} @{if({dblquote}${REVISION}{dblquote} !=  {dblquote}${ISSUE_DATE}{dblquote}, {dblquote}(${ISSUE_DATE}){dblquote}, {dblquote}{dblquote})}"
-		(at 7.75 8.25 0)
-		(layer "F.Fab")
+		(at 49 45 0)
+		(layer "Cmts.User")
 		(effects
 			(font
@@
 	(gr_text "280 x 380 -> 200 x 320"
 		(locked yes)
-		(at 212.5 373.75 0)
-		(layer "F.Fab")
+		(at 179.75 360.75 0)
+		(layer "Cmts.User")
 		(effects
 			(font
@@
 		)
 	)
+	(gr_text "1:1 please. No changes. Do NOT remove any fiducials. Thanks!"
+		(at 140 15 0)
+		(layer "Cmts.User")
+		(effects
+			(font
+				(size 4 4)
+				(thickness 0.6)
+				(bold yes)
+			)
+			(justify top)
+		)
+	)

Commit message: Update LDO
Other:
- board text removed: "1:1 please. No changes. Do NOT remove any fiducials. Thanks!"
Changed lines of the file:
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@@
 	(paper "User" 280 380)
 	(title_block
-		(date "2026-07-18")
-		(rev "2026-07-18")
+		(date "2026-08-21")
+		(rev "2026-08-21")
 	)
 	(layers
@@
 		(grid_origin 40 350)
 		(pcbplotparams
-			(layerselection 0x00000000_00000000_55555555_555d7500)
+			(layerselection 0x00000000_00000000_55555555_55557500)
 			(plot_on_all_layers_selection 0x00000000_00000000_00000000_00000000)
 			(disableapertmacros no)
@@
 		)
 	)
-	(gr_text "1:1 please. No changes. Do NOT remove any fiducials. Thanks!"
-		(at 140 15 0)
-		(layer "Cmts.User")
-		(effects
-			(font
-				(size 4 4)
-				(thickness 0.6)
-				(bold yes)
-			)
-			(justify top)
-		)
-	)
