File: template/stencil/stencil.kicad_sch (KiCad schematic)
At the start: 3 parts

Commit message: Update stencil template
Parts:
- FID101, FID102, FID103: value Fiducial -> Fiducial_Paste
Other:
- moved on the sheet: FID101, FID102, FID103
Changed lines of the file:
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@@
 	(title_block
 		(title "stencil")
-		(date "2026-01-10")
+		(date "2026-02-10")
 		(company "Versio Duo")
 	)
 	(symbol
 		(lib_id "V2_Mechanical:Fiducial_Paste")
-		(at 120.65 264.16 0)
+		(at 184.15 255.27 0)
 		(unit 1)
-		(exclude_from_sim yes)
+		(exclude_from_sim no)
 		(in_bom no)
 		(on_board yes)
 		(dnp no)
 		(property "Reference" "FID101"
-			(at 118.11 257.81 0)
+			(at 187.198 255.27 0)
 			(effects
 				(font
@@
 			)
 		)
-		(property "Value" "Fiducial"
-			(at 120.65 260.35 0)
-			(effects
-				(font
-					(size 1.27 1.27)
-				)
+		(property "Value" "Fiducial_Paste"
+			(at 184.15 251.46 0)
+			(effects
+				(font
+					(size 1.27 1.27)
+				)
+				(hide yes)
 			)
 		)
 		(property "Footprint" "V2_Fiducial:Fiducial_0.5mm_Mask1mm_Paste"
-			(at 120.65 269.24 0)
+			(at 184.15 260.35 0)
 			(effects
 				(font
@@
 		)
 		(property "Datasheet" ""
-			(at 120.65 264.16 0)
+			(at 184.15 255.27 0)
 			(effects
 				(font
@@
 		)
 		(property "Description" "Fiducial Marker"
-			(at 120.65 264.16 0)
+			(at 184.15 255.27 0)
 			(effects
 				(font
@@
 	(symbol
 		(lib_id "V2_Mechanical:Fiducial_Paste")
-		(at 138.43 264.16 0)
+		(at 184.15 265.43 0)
 		(unit 1)
-		(exclude_from_sim yes)
+		(exclude_from_sim no)
 		(in_bom no)
 		(on_board yes)
 		(dnp no)
 		(property "Reference" "FID103"
-			(at 135.89 257.81 0)
+			(at 187.198 265.43 0)
 			(effects
 				(font
@@
 			)
 		)
-		(property "Value" "Fiducial"
-			(at 139.7 260.35 0)
-			(effects
-				(font
-					(size 1.27 1.27)
-				)
+		(property "Value" "Fiducial_Paste"
+			(at 185.42 261.62 0)
+			(effects
+				(font
+					(size 1.27 1.27)
+				)
+				(hide yes)
 			)
 		)
 		(property "Footprint" "V2_Fiducial:Fiducial_0.5mm_Mask1mm_Paste"
-			(at 138.43 269.24 0)
+			(at 184.15 270.51 0)
 			(effects
 				(font
@@
 		)
 		(property "Datasheet" ""
-			(at 138.43 264.16 0)
+			(at 184.15 265.43 0)
 			(effects
 				(font
@@
 		)
 		(property "Description" "Fiducial Marker"
-			(at 138.43 264.16 0)
+			(at 184.15 265.43 0)
 			(effects
 				(font
@@
 	(symbol
 		(lib_id "V2_Mechanical:Fiducial_Paste")
-		(at 129.54 264.16 0)
+		(at 184.15 260.35 0)
 		(unit 1)
-		(exclude_from_sim yes)
+		(exclude_from_sim no)
 		(in_bom no)
 		(on_board yes)
 		(dnp no)
 		(property "Reference" "FID102"
-			(at 127 257.81 0)
+			(at 187.198 260.35 0)
 			(effects
 				(font
@@
 			)
 		)
-		(property "Value" "Fiducial"
-			(at 129.54 260.35 0)
-			(effects
-				(font
-					(size 1.27 1.27)
-				)
+		(property "Value" "Fiducial_Paste"
+			(at 184.15 256.54 0)
+			(effects
+				(font
+					(size 1.27 1.27)
+				)
+				(hide yes)
 			)
 		)
 		(property "Footprint" "V2_Fiducial:Fiducial_0.5mm_Mask1mm_Paste"
-			(at 129.54 269.24 0)
+			(at 184.15 265.43 0)
 			(effects
 				(font
@@
 		)
 		(property "Datasheet" ""
-			(at 129.54 264.16 0)
+			(at 184.15 260.35 0)
 			(effects
 				(font
@@
 		)
 		(property "Description" "Fiducial Marker"
-			(at 129.54 264.16 0)
+			(at 184.15 260.35 0)
 			(effects
 				(font
@@
 	)
 	(embedded_fonts no)
+	(embedded_files
+		(file
+			(name "V2_A4.kicad_wks")
+			(type worksheet)
+			(data |KLUv/WBhBk0QALbYTiEQtRsmZc5q276ayLS71D6kxbkmoTeIJM7lAHtEAMAAxQFGAD8ARQCbvIHa
+				a/wrVHSazXnPhvzar1BNtH1kxRf5EwCAQPh5F+e0kJq0nmtfKDvj37Jf3xQUlFKqztoXWzE7iAAI
+				iJ6Q5m2d9RAC9jcPPWe/GXf/9ewpPR3+uPbv7bdzvr37wXlr2X8dBHFXu7Z3HUG7Kvrz9qKU7eB2
+				v/MM4n/Mhfg5G5sn7WsDTS2mA1WyssZDsy4YdpEGzfD8Ny+85JzH7H+961FjX/x0qtq0MdaqJ8dx
+				k1KAwF+soV3VFnEoqewX+XNfTaqqPatRlLsbgcKhzs5+29sEzSaWRPZ4txDEjpmZNCoSiiMhaUwy
+				y4Jg3oe5pmhPRSS7MtJAerbfnYNNgaEkuCg6oVzYhbEsF1vRgtxS55zTIVig4URjFFJTI1qYFNIB
+				YESmRusYYvaiF0uSUdhu1Q2lFiOgdmN7VvaH2oWyw9MQXRuZtQQQoIsxFn2ldtnpQiUNa0HvDQCK
+				f/XTisCgEJQEXe/if4EJsakkqj8BMmGAU+ZM/AG8LSEJMfgkOKfSKPhw4rD3ZHfmNZYNfDMigEPJ
+				EBoIDghtm1kJ8BAQ8xyGdkOuFQy33sishFt8DZNX4uNRXJZ5hBy746RJaNtgbfyB613d0dov6Cdg
+				iUQT9BXkf9EiYDuODpB6gKkC|
+			)
+			(checksum "0A61268C685EAF945CA2EA8187370BD3")
+		)
+	)
 )
