File: template/default/default.kicad_sch (KiCad schematic)
At the start: 0 parts

Commit message: Update default 4-layer stackup
Other:
- company: Versio duo -> Versio Duo
Changed lines of the file:
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@@
 	(title_block
 		(title "default")
-		(date "2026-04-23")
-		(rev "2026-04-23")
-		(company "Versio duo")
+		(date "2026-05-30")
+		(rev "2026-05-30")
+		(company "Versio Duo")
 	)
 	(sheet_instances
